File: lab4/555 Circuit/ee210.kicad_pcb (KiCad board)
At the start: 2 copper layers, 63.5 x 48.3 mm, 10 parts, among them J1 Conn_01x02_Male, U1 NE555D

Commit message: lab7
Other:
- board size 63.5 x 48.3 mm -> 40.6 x 48.3 mm
- board text added: "EE 201 555 Timer"
- board text added: "Lucas Elroy"
