File: lab4/LED Circuit/LED.kicad_sch (KiCad schematic)
At the start: 7 parts, among them SW1 Conn_01x02_Male, SW1 SW_SPDT

Commit message: “tes”
Parts:
- removed SW1: Conn_01x02_Male, symbol Connector:Conn_01x02_Male
- C1: footprint (none) -> Capacitor_THT:C_Radial_D5.0mm_H5.0mm_P2.00mm
- D1: footprint (none) -> LED_THT:LED_D5.0mm
- R1, R2: footprint (none) -> Resistor_THT:R_Axial_DIN0516_L15.5mm_D5.0mm_P20.32mm_Horizontal
- SW1: footprint (none) -> Button_Switch_THT:SW_E-Switch_EG1224_SPDT_Angled
- V1: footprint (none) -> Connector_JST:JST_PH_B2B-PH-K_1x02_P2.00mm_Vertical
Connections:
- net at SW1.3 (C): now also C1.1, R1.2
Other:
- moved on the sheet: R2, SW1
Changed lines of the file:
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@@
   (junction (at 116.84 127) (diameter 0) (color 0 0 0 0)
   )
-  (wire (pts (xy 88.9 101.6) (xy 92.71 101.6))
+  (junction (at 116.84 102.87) (diameter 0) (color 0 0 0 0)
+  )
+  (wire (pts (xy 116.84 102.87) (xy 116.84 110.49))
     (stroke (width 0) (type default) (color 0 0 0 0))
   )
-  (wire (pts (xy 129.54 102.87) (xy 142.24 102.87))
-    (stroke (width 0) (type default) (color 0 0 0 0))
-  )
-  (wire (pts (xy 116.84 110.49) (xy 116.84 104.14))
+  (wire (pts (xy 88.9 100.33) (xy 92.71 100.33))
     (stroke (width 0) (type default) (color 0 0 0 0))
   )
@@
     (stroke (width 0) (type default) (color 0 0 0 0))
   )
-  (wire (pts (xy 124.46 102.87) (xy 120.65 102.87))
-    (stroke (width 0) (type default) (color 0 0 0 0))
-  )
   (wire (pts (xy 142.24 110.49) (xy 142.24 115.57))
     (stroke (width 0) (type default) (color 0 0 0 0))
   )
-  (wire (pts (xy 88.9 110.49) (xy 88.9 101.6))
+  (wire (pts (xy 88.9 100.33) (xy 88.9 110.49))
+    (stroke (width 0) (type default) (color 0 0 0 0))
+  )
+  (wire (pts (xy 116.84 102.87) (xy 142.24 102.87))
     (stroke (width 0) (type default) (color 0 0 0 0))
   )
   (wire (pts (xy 142.24 127) (xy 116.84 127))
-    (stroke (width 0) (type default) (color 0 0 0 0))
-  )
-  (wire (pts (xy 120.65 99.06) (xy 124.46 100.33))
     (stroke (width 0) (type default) (color 0 0 0 0))
   )
@@
     (stroke (width 0) (type default) (color 0 0 0 0))
   )
-  (wire (pts (xy 116.84 104.14) (xy 118.11 104.14))
-    (stroke (width 0) (type default) (color 0 0 0 0))
-  )
-  (wire (pts (xy 100.33 101.6) (xy 110.49 101.6))
-    (stroke (width 0) (type default) (color 0 0 0 0))
-  )
-  (wire (pts (xy 120.65 102.87) (xy 120.65 104.14))
+  (wire (pts (xy 100.33 100.33) (xy 106.68 100.33))
     (stroke (width 0) (type default) (color 0 0 0 0))
   )
@@
       (effects (font (size 1.27 1.27)) (justify right) hide)
     )
-    (property "Footprint" "" (id 2) (at 142.24 119.38 0)
+    (property "Footprint" "LED_THT:LED_D5.0mm" (id 2) (at 142.24 119.38 0)
       (effects (font (size 1.27 1.27)) hide)
     )
@@
     (pin "2")
   )
-  (symbol (lib_id "Connector:Conn_01x02_Male") (at 129.54 102.87 180) (unit 1)
+  (symbol (lib_id "Device:R") (at 96.52 100.33 90) (unit 1)
     (in_bom yes) (on_board yes) (fields_autoplaced)
-    (property "Reference" "SW1" (id 0) (at 128.905 107.95 0)
+    (property "Reference" "R2" (id 0) (at 96.52 93.98 90))
+    (property "Value" "2.2k" (id 1) (at 96.52 96.52 90))
+    (property "Footprint" "Resistor_THT:R_Axial_DIN0516_L15.5mm_D5.0mm_P20.32mm_Horizontal" (id 2) (at 96.52 102.108 90)
       (effects (font (size 1.27 1.27)) hide)
     )
-    (property "Value" "Conn_01x02_Male" (id 1) (at 128.905 105.41 0)
-      (effects (font (size 1.27 1.27)) hide)
-    )
-    (property "Footprint" "" (id 2) (at 129.54 102.87 0)
-      (effects (font (size 1.27 1.27)) hide)
-    )
-    (property "Datasheet" "~" (id 3) (at 129.54 102.87 0)
-      (effects (font (size 1.27 1.27)) hide)
-    )
-    (pin "1")
-    (pin "2")
-  )
-  (symbol (lib_id "Device:R") (at 96.52 101.6 90) (unit 1)
-    (in_bom yes) (on_board yes) (fields_autoplaced)
-    (property "Reference" "R2" (id 0) (at 96.52 95.25 90))
-    (property "Value" "2.2k" (id 1) (at 96.52 97.79 90))
-    (property "Footprint" "" (id 2) (at 96.52 103.378 90)
-      (effects (font (size 1.27 1.27)) hide)
-    )
-    (property "Datasheet" "~" (id 3) (at 96.52 101.6 0)
+    (property "Datasheet" "~" (id 3) (at 96.52 100.33 0)
       (effects (font (size 1.27 1.27)) hide)
     )
@@
       (effects (font (size 1.27 1.27)) (justify left))
     )
-    (property "Footprint" "" (id 2) (at 117.8052 118.11 0)
+    (property "Footprint" "Capacitor_THT:C_Radial_D5.0mm_H5.0mm_P2.00mm" (id 2) (at 117.8052 118.11 0)
       (effects (font (size 1.27 1.27)) hide)
     )
@@
       (effects (font (size 1.27 1.27)) (justify left))
     )
-    (property "Footprint" "" (id 2) (at 88.9 114.046 90)
+    (property "Footprint" "Connector_JST:JST_PH_B2B-PH-K_1x02_P2.00mm_Vertical" (id 2) (at 88.9 114.046 90)
       (effects (font (size 1.27 1.27)) hide)
     )
@@
       (effects (font (size 1.27 1.27)) (justify right))
     )
-    (property "Footprint" "" (id 2) (at 144.018 106.68 90)
+    (property "Footprint" "Resistor_THT:R_Axial_DIN0516_L15.5mm_D5.0mm_P20.32mm_Horizontal" (id 2) (at 144.018 106.68 90)
       (effects (font (size 1.27 1.27)) hide)
     )
@@
     (pin "2")
   )
-  (symbol (lib_id "Switch:SW_SPDT") (at 115.57 101.6 0) (unit 1)
+  (symbol (lib_id "Switch:SW_SPDT") (at 111.76 100.33 0) (unit 1)
     (in_bom yes) (on_board yes) (fields_autoplaced)
-    (property "Reference" "SW1" (id 0) (at 115.57 93.98 0))
-    (property "Value" "SW_SPDT" (id 1) (at 115.57 96.52 0)
+    (property "Reference" "SW1" (id 0) (at 111.76 95.25 0))
+    (property "Value" "SW_SPDT" (id 1) (at 111.76 95.25 0)
       (effects (font (size 1.27 1.27)) hide)
     )
-    (property "Footprint" "" (id 2) (at 115.57 101.6 0)
+    (property "Footprint" "Button_Switch_THT:SW_E-Switch_EG1224_SPDT_Angled" (id 2) (at 111.76 100.33 0)
       (effects (font (size 1.27 1.27)) hide)
     )
-    (property "Datasheet" "~" (id 3) (at 115.57 101.6 0)
+    (property "Datasheet" "~" (id 3) (at 111.76 100.33 0)
       (effects (font (size 1.27 1.27)) hide)
     )
@@
   (symbol_instances
     (path "/53478b23-aca6-44c6-a5b1-997a1fc94e3f"
-      (reference "C1") (unit 1) (value "4.7uF") (footprint "")
+      (reference "C1") (unit 1) (value "4.7uF") (footprint "Capacitor_THT:C_Radial_D5.0mm_H5.0mm_P2.00mm")
     )
     (path "/1723fede-9f67-4a50-b001-487722d652ff"
-      (reference "D1") (unit 1) (value "LED") (footprint "")
+      (reference "D1") (unit 1) (value "LED") (footprint "LED_THT:LED_D5.0mm")
     )
     (path "/b7315d5d-efee-4564-a4af-2b44108fd641"
-      (reference "R1") (unit 1) (value "20k") (footprint "")
+      (reference "R1") (unit 1) (value "20k") (footprint "Resistor_THT:R_Axial_DIN0516_L15.5mm_D5.0mm_P20.32mm_Horizontal")
     )
     (path "/4defab3c-c616-4817-acf9-b97ebec0bb74"
-      (reference "R2") (unit 1) (value "2.2k") (footprint "")
-    )
-    (path "/407f0c9a-7540-4f9f-a4f1-cc69dcdf8fa8"
-      (reference "SW1") (unit 1) (value "Conn_01x02_Male") (footprint "")
+      (reference "R2") (unit 1) (value "2.2k") (footprint "Resistor_THT:R_Axial_DIN0516_L15.5mm_D5.0mm_P20.32mm_Horizontal")
     )
     (path "/faa6a489-b5b8-455f-95ad-ae97b754314f"
-      (reference "SW1") (unit 1) (value "SW_SPDT") (footprint "")
+      (reference "SW1") (unit 1) (value "SW_SPDT") (footprint "Button_Switch_THT:SW_E-Switch_EG1224_SPDT_Angled")
     )
     (path "/638a47ee-467c-4ba3-bdb1-2e578e88a21a"
-      (reference "V1") (unit 1) (value "9V") (footprint "")
+      (reference "V1") (unit 1) (value "9V") (footprint "Connector_JST:JST_PH_B2B-PH-K_1x02_P2.00mm_Vertical")
     )
   )
